File: hikari.kicad_sch (KiCad schematic)
At the start: 2 parts, among them SW1 Switch, SW2 Switch

Commit message: did most of todo items
Parts:
- added CN2: 1x3, symbol pin_headers:1x3
- added R16: 10k, SMT:0603, symbol generic:R
- SW1: value Switch -> LS12W3-T; footprint (none) -> buttons:LS12W3-T; symbol generic:Switch -> switches:LS12W3-T; Digi-Key (none) -> 1642-LS12W3-TCT-ND
- SW2: value Switch -> JS102011SAQN; footprint (none) -> buttons:JS102011SAQN; symbol generic:Switch -> switches:JS102011SAQN; Digi-Key (none) -> 401-1999-1-ND
Connections:
- net GND: now also SW1.1, CN2.3, R16.1; no longer SW1.~, SW2.~
- net MCU/Button_1: now also SW1.2; no longer SW1.~
- removed net MCU/Button_2: SW2.~
- new net: SW2.3, SW2.4
- new net 5V: CN2.1, SW2.1
- new net MCU/LED_strip: CN2.2
- new net Power supply/Enable: R16.2, SW2.2
Other:
- sheet MCU ports: added LED_strip; removed Button_2
- sheet Power supply ports: added Enable; removed none
