File: hikari.kicad_sch (KiCad schematic)
At the start: 4 parts, among them CN2 1x3, SW1 LS12W3-T, SW2 JS102011SAQN

Commit message: added Digi-Key part numbers to BOM
Parts:
- R16: Digi-Key (none) -> 13-RC0603JR-1010KLCT-ND
Changed lines of the file:
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@@
+      (effects (font (size 1.27 1.27)) hide)
+    )
+    (property "Digi-Key" "13-RC0603JR-1010KLCT-ND" (at 91.44 71.12 0)
       (effects (font (size 1.27 1.27)) hide)
     )
