File: LED.kicad_sch (KiCad schematic)
At the start: 6 parts, among them IC1 PAM2804AAB010

Commit message: fixed power symbols from showing up in BOM
Parts:
- C1, C2: footprint SMT:0805 -> SMT:0603
Changed lines of the file:
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@@
       (effects (font (size 1.27 1.27)) (justify left top))
     )
-    (property "Footprint" "SMT:0805" (at 124.46 99.06 0)
+    (property "Footprint" "SMT:0603" (at 124.46 99.06 0)
       (effects (font (size 1.27 1.27)) hide)
     )
@@
   (symbol (lib_id "generic:GND") (at 172.72 109.22 0) (unit 1)
     (in_bom yes) (on_board yes) (dnp no) (fields_autoplaced)
-    (property "Reference" "#GND04" (at 176.53 107.95 0)
+    (property "Reference" "#GND?" (at 176.53 107.95 0)
       (effects (font (size 1.27 1.27)) hide)
     )
@@
       (project "hikari"
         (path "/020af8ab-593e-45b9-b2cd-8db025796961/aa80c023-a405-4836-a45d-48fe501d72e6"
-          (reference "#GND04") (unit 1)
-        )
-        (path "/020af8ab-593e-45b9-b2cd-8db025796961/4047ad27-abaf-44fc-8fae-330cc49c4e32"
-          (reference "#GND08") (unit 1)
-        )
-        (path "/020af8ab-593e-45b9-b2cd-8db025796961/1271e14e-21a7-43a9-b754-008b9cfd2c5b"
-          (reference "#GND012") (unit 1)
-        )
-        (path "/020af8ab-593e-45b9-b2cd-8db025796961/78613248-b522-4bfb-a044-b4a58ad1b605"
-          (reference "#GND016") (unit 1)
+          (reference "#GND?") (unit 1)
+        )
+        (path "/020af8ab-593e-45b9-b2cd-8db025796961/4047ad27-abaf-44fc-8fae-330cc49c4e32"
+          (reference "#GND?") (unit 1)
+        )
+        (path "/020af8ab-593e-45b9-b2cd-8db025796961/1271e14e-21a7-43a9-b754-008b9cfd2c5b"
+          (reference "#GND?") (unit 1)
+        )
+        (path "/020af8ab-593e-45b9-b2cd-8db025796961/78613248-b522-4bfb-a044-b4a58ad1b605"
+          (reference "#GND?") (unit 1)
         )
       )
@@
   (symbol (lib_id "generic:GND") (at 134.62 109.22 0) (unit 1)
     (in_bom yes) (on_board yes) (dnp no) (fields_autoplaced)
-    (property "Reference" "#GND02" (at 138.43 107.95 0)
+    (property "Reference" "#GND?" (at 138.43 107.95 0)
       (effects (font (size 1.27 1.27)) hide)
     )
@@
       (project "hikari"
         (path "/020af8ab-593e-45b9-b2cd-8db025796961/aa80c023-a405-4836-a45d-48fe501d72e6"
-          (reference "#GND02") (unit 1)
-        )
-        (path "/020af8ab-593e-45b9-b2cd-8db025796961/4047ad27-abaf-44fc-8fae-330cc49c4e32"
-          (reference "#GND06") (unit 1)
-        )
-        (path "/020af8ab-593e-45b9-b2cd-8db025796961/1271e14e-21a7-43a9-b754-008b9cfd2c5b"
-          (reference "#GND010") (unit 1)
-        )
-        (path "/020af8ab-593e-45b9-b2cd-8db025796961/78613248-b522-4bfb-a044-b4a58ad1b605"
-          (reference "#GND014") (unit 1)
+          (reference "#GND?") (unit 1)
+        )
+        (path "/020af8ab-593e-45b9-b2cd-8db025796961/4047ad27-abaf-44fc-8fae-330cc49c4e32"
+          (reference "#GND?") (unit 1)
+        )
+        (path "/020af8ab-593e-45b9-b2cd-8db025796961/1271e14e-21a7-43a9-b754-008b9cfd2c5b"
+          (reference "#GND?") (unit 1)
+        )
+        (path "/020af8ab-593e-45b9-b2cd-8db025796961/78613248-b522-4bfb-a044-b4a58ad1b605"
+          (reference "#GND?") (unit 1)
         )
       )
@@
   (symbol (lib_id "generic:GND") (at 162.56 109.22 0) (unit 1)
     (in_bom yes) (on_board yes) (dnp no) (fields_autoplaced)
-    (property "Reference" "#GND03" (at 166.37 107.95 0)
+    (property "Reference" "#GND?" (at 166.37 107.95 0)
       (effects (font (size 1.27 1.27)) hide)
     )
@@
       (project "hikari"
         (path "/020af8ab-593e-45b9-b2cd-8db025796961/aa80c023-a405-4836-a45d-48fe501d72e6"
-          (reference "#GND03") (unit 1)
-        )
-        (path "/020af8ab-593e-45b9-b2cd-8db025796961/4047ad27-abaf-44fc-8fae-330cc49c4e32"
-          (reference "#GND07") (unit 1)
-        )
-        (path "/020af8ab-593e-45b9-b2cd-8db025796961/1271e14e-21a7-43a9-b754-008b9cfd2c5b"
-          (reference "#GND011") (unit 1)
-        )
-        (path "/020af8ab-593e-45b9-b2cd-8db025796961/78613248-b522-4bfb-a044-b4a58ad1b605"
-          (reference "#GND015") (unit 1)
+          (reference "#GND?") (unit 1)
+        )
+        (path "/020af8ab-593e-45b9-b2cd-8db025796961/4047ad27-abaf-44fc-8fae-330cc49c4e32"
+          (reference "#GND?") (unit 1)
+        )
+        (path "/020af8ab-593e-45b9-b2cd-8db025796961/1271e14e-21a7-43a9-b754-008b9cfd2c5b"
+          (reference "#GND?") (unit 1)
+        )
+        (path "/020af8ab-593e-45b9-b2cd-8db025796961/78613248-b522-4bfb-a044-b4a58ad1b605"
+          (reference "#GND?") (unit 1)
         )
       )
@@
   (symbol (lib_id "generic:GND") (at 124.46 109.22 0) (unit 1)
     (in_bom yes) (on_board yes) (dnp no) (fields_autoplaced)
-    (property "Reference" "#GND01" (at 128.27 107.95 0)
+    (property "Reference" "#GND?" (at 128.27 107.95 0)
       (effects (font (size 1.27 1.27)) hide)
     )
@@
       (project "hikari"
         (path "/020af8ab-593e-45b9-b2cd-8db025796961/aa80c023-a405-4836-a45d-48fe501d72e6"
-          (reference "#GND01") (unit 1)
-        )
-        (path "/020af8ab-593e-45b9-b2cd-8db025796961/4047ad27-abaf-44fc-8fae-330cc49c4e32"
-          (reference "#GND05") (unit 1)
-        )
-        (path "/020af8ab-593e-45b9-b2cd-8db025796961/1271e14e-21a7-43a9-b754-008b9cfd2c5b"
-          (reference "#GND09") (unit 1)
-        )
-        (path "/020af8ab-593e-45b9-b2cd-8db025796961/78613248-b522-4bfb-a044-b4a58ad1b605"
-          (reference "#GND013") (unit 1)
+          (reference "#GND?") (unit 1)
+        )
+        (path "/020af8ab-593e-45b9-b2cd-8db025796961/4047ad27-abaf-44fc-8fae-330cc49c4e32"
+          (reference "#GND?") (unit 1)
+        )
+        (path "/020af8ab-593e-45b9-b2cd-8db025796961/1271e14e-21a7-43a9-b754-008b9cfd2c5b"
+          (reference "#GND?") (unit 1)
+        )
+        (path "/020af8ab-593e-45b9-b2cd-8db025796961/78613248-b522-4bfb-a044-b4a58ad1b605"
+          (reference "#GND?") (unit 1)
         )
       )
@@
       (effects (font (size 1.27 1.27)) (justify left top))
     )
-    (property "Footprint" "SMT:0805" (at 172.72 99.06 0)
-      (effects (font (size 1.27 1.27)) hide)
-    )
+    (property "Footprint" "SMT:0603" (at 172.72 99.06 0)
+      (effects (font (size 1.27 1.27)) hide)
+    )

Commit message: added Digi-Key part numbers to BOM
Parts:
- C1, C2: Digi-Key (none) -> 1276-1119-1-ND
- L1: Digi-Key (none) -> 308-1590-1-ND
- R1: Digi-Key (none) -> 273-KDV06FR300ETCT-ND
Changed lines of the file:
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@@
+      (effects (font (size 1.27 1.27)) hide)
+    )
+    (property "Digi-Key" "273-KDV06FR300ETCT-ND" (at 162.56 101.6 0)
       (effects (font (size 1.27 1.27)) hide)
     )
@@
       (effects (font (size 1.27 1.27)) hide)
     )
+    (property "Digi-Key" "1276-1119-1-ND" (at 124.46 96.52 0)
+      (effects (font (size 1.27 1.27)) hide)
+    )
     (pin "1")
     (pin "2")
@@
     )
     (property "Datasheet" "" (at 157.48 86.36 0)
+      (effects (font (size 1.27 1.27)) hide)
+    )
+    (property "Digi-Key" "308-1590-1-ND" (at 157.48 86.36 0)
       (effects (font (size 1.27 1.27)) hide)
     )
@@
       (effects (font (size 1.27 1.27)) hide)
     )
+    (property "Digi-Key" "1276-1119-1-ND" (at 172.72 96.52 0)
+      (effects (font (size 1.27 1.27)) hide)
+    )
