File: USB.kicad_sch (KiCad schematic)
At the start: 7 parts, among them CN1 USB-C, IC6 CH340G, x1 xtal_osc

Commit message: did most of todo items
Parts:
- added R13, R15: 5k1, SMT:0603, symbol generic:R
- x1: value xtal_osc -> 12MHZ; footprint (none) -> xtal:3.2x2.5CXO; symbol oscillators:xtal_osc -> oscillators:RH100-12.000-18-2020-EXT-TR; Digi-Key (none) -> 2151-RH100-12.000-18-2020-EXT-TRCT-ND
Connections:
- net GND: now also R13.1, R15.1
- net DP: now reaches CN1.A6 (D1P), IC6.5 (UD+)
- net DP: now also CN1.B6 (DP2)
- net DN: now reaches CN1.A7 (D1N), IC6.6 (UD-)
- net DN: now also CN1.B7 (DN2)
- net at CN1.A5 (CC1): now also R13.2
- net at CN1.B5 (CC2): now also R15.2
Changed lines of the file:
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@@
+    (stroke (width 0) (type default))
+  )
+  (wire (pts (xy 83.82 101.6) (xy 91.44 101.6))
     (stroke (width 0) (type default))
   )
@@
     (stroke (width 0) (type default))
   )
+  (wire (pts (xy 83.82 111.76) (xy 83.82 109.22))
+    (stroke (width 0) (type default))
+  )
   (wire (pts (xy 143.51 113.03) (xy 147.32 113.03))
     (stroke (width 0) (type default))
@@
     (stroke (width 0) (type default))
   )
+  (wire (pts (xy 111.76 93.98) (xy 119.38 93.98))
+    (stroke (width 0) (type default))
+  )
   (wire (pts (xy 147.32 106.68) (xy 157.48 106.68))
     (stroke (width 0) (type default))
@@
     (stroke (width 0) (type default))
   )
+  (wire (pts (xy 88.9 96.52) (xy 91.44 96.52))
+    (stroke (width 0) (type default))
+  )
   (wire (pts (xy 177.8 91.44) (xy 180.34 91.44))
     (stroke (width 0) (type default))
@@
     (stroke (width 0) (type default))
   )
-  (wire (pts (xy 88.9 109.22) (xy 88.9 106.68))
+  (wire (pts (xy 88.9 111.76) (xy 88.9 106.68))
+    (stroke (width 0) (type default))
+  )
+  (wire (pts (xy 88.9 99.06) (xy 91.44 99.06))
     (stroke (width 0) (type default))
   )
@@
     (stroke (width 0) (type default))
   )
+  (wire (pts (xy 119.38 93.98) (xy 119.38 104.14))
+    (stroke (width 0) (type default))
+  )
   (wire (pts (xy 88.9 106.68) (xy 91.44 106.68))
     (stroke (width 0) (type default))
@@
     (stroke (width 0) (type default))
   )
+  (wire (pts (xy 119.38 109.22) (xy 119.38 111.76))
+    (stroke (width 0) (type default))
+  )
   (wire (pts (xy 99.06 116.84) (xy 99.06 119.38))
     (stroke (width 0) (type default))
@@
     (stroke (width 0) (type default))
   )
-  (wire (pts (xy 114.3 106.68) (xy 114.3 109.22))
+  (wire (pts (xy 114.3 106.68) (xy 114.3 111.76))
     (stroke (width 0) (type default))
   )
@@
     (stroke (width 0) (type default))
   )
+  (wire (pts (xy 83.82 104.14) (xy 83.82 101.6))
+    (stroke (width 0) (type default))
+  )
   (wire (pts (xy 114.3 88.9) (xy 114.3 78.74))
     (stroke (width 0) (type default))
@@
   (wire (pts (xy 154.94 109.22) (xy 154.94 121.92))
     (stroke (width 0) (type default))
+  )
+  (label "DN" (at 114.3 99.06 0) (fields_autoplaced)
+    (effects (font (size 1.27 1.27)) (justify left bottom))
+  )
+  (label "DP" (at 88.9 99.06 0) (fields_autoplaced)
+    (effects (font (size 1.27 1.27)) (justify left bottom))
+  )
+  (label "DN" (at 88.9 96.52 0) (fields_autoplaced)
+    (effects (font (size 1.27 1.27)) (justify left bottom))
+  )
+  (label "DP" (at 114.3 96.52 0) (fields_autoplaced)
+    (effects (font (size 1.27 1.27)) (justify left bottom))
   )
   (hierarchical_label "V_USB" (shape output) (at 128.27 76.2 0) (fields_autoplaced)
@@
     )
   )
+  (symbol (lib_id "generic:R") (at 119.38 106.68 90) (unit 1)
+    (in_bom yes) (on_board yes) (dnp no)
+    (property "Reference" "R13" (at 120.65 106.68 90)
+      (effects (font (size 1.27 1.27)) (justify right top))
+    )
+    (property "Value" "5k1" (at 120.65 106.68 90)
+      (effects (font (size 1.27 1.27)) (justify right bottom))
+    )
+    (property "Footprint" "SMT:0603" (at 120.015 109.22 0)
+      (effects (font (size 1.27 1.27)) hide)
+    )
+    (property "Datasheet" "" (at 119.38 106.68 0)
+      (effects (font (size 1.27 1.27)) hide)
+    )
+    (pin "1")
+    (pin "2")
+    (instances
+      (project "hikari"
+        (path "/020af8ab-593e-45b9-b2cd-8db025796961/bb941b2b-0b73-4110-b4b0-cdc102f480d3"
+          (reference "R13") (unit 1)
+        )
+      )
+    )
+  )
   (symbol (lib_id "generic:C") (at 132.08 86.36 0) (unit 1)
     (in_bom yes) (on_board yes) (dnp no)
@@
     )
   )
-  (symbol (lib_id "generic:GND") (at 88.9 109.22 0) (unit 1)
-    (in_bom yes) (on_board yes) (dnp no) (fields_autoplaced)
-    (property "Reference" "#GND05" (at 92.71 107.95 0)
-      (effects (font (size 1.27 1.27)) hide)
-    )
-    (property "Value" "GND" (at 92.71 109.22 0)
-      (effects (font (size 1.27 1.27)) hide)
-    )
-    (property "Footprint" "" (at 88.9 109.22 0)
-      (effects (font (size 1.27 1.27)) hide)
-    )
-    (property "Datasheet" "" (at 88.9 109.22 0)
+  (symbol (lib_id "generic:GND") (at 88.9 111.76 0) (unit 1)
+    (in_bom yes) (on_board yes) (dnp no) (fields_autoplaced)
+    (property "Reference" "#GND05" (at 92.71 110.49 0)
+      (effects (font (size 1.27 1.27)) hide)
+    )
+    (property "Value" "GND" (at 92.71 111.76 0)
+      (effects (font (size 1.27 1.27)) hide)
+    )
+    (property "Footprint" "" (at 88.9 111.76 0)
+      (effects (font (size 1.27 1.27)) hide)
+    )
+    (property "Datasheet" "" (at 88.9 111.76 0)
       (effects (font (size 1.27 1.27)) hide)
     )
@@
     )
   )
-  (symbol (lib_id "generic:GND") (at 114.3 109.22 0) (unit 1)
-    (in_bom yes) (on_board yes) (dnp no) (fields_autoplaced)
-    (property "Reference" "#GND0124" (at 118.11 107.95 0)
-      (effects (font (size 1.27 1.27)) hide)
-    )
-    (property "Value" "GND" (at 118.11 109.22 0)
-      (effects (font (size 1.27 1.27)) hide)
-    )
-    (property "Footprint" "" (at 114.3 109.22 0)
-      (effects (font (size 1.27 1.27)) hide)
-    )
-    (property "Datasheet" "" (at 114.3 109.22 0)
+  (symbol (lib_id "generic:GND") (at 114.3 111.76 0) (unit 1)
+    (in_bom yes) (on_board yes) (dnp no) (fields_autoplaced)
+    (property "Reference" "#GND0124" (at 118.11 110.49 0)
+      (effects (font (size 1.27 1.27)) hide)
+    )
+    (property "Value" "GND" (at 118.11 111.76 0)
+      (effects (font (size 1.27 1.27)) hide)
+    )
+    (property "Footprint" "" (at 114.3 111.76 0)
+      (effects (font (size 1.27 1.27)) hide)
+    )
+    (property "Datasheet" "" (at 114.3 111.76 0)
       (effects (font (size 1.27 1.27)) hide)
     )
@@
     )
   )
+  (symbol (lib_id "generic:GND") (at 119.38 111.76 0) (unit 1)
+    (in_bom yes) (on_board yes) (dnp no) (fields_autoplaced)
+    (property "Reference" "#GND06" (at 123.19 110.49 0)
+      (effects (font (size 1.27 1.27)) hide)
+    )
+    (property "Value" "GND" (at 123.19 111.76 0)
+      (effects (font (size 1.27 1.27)) hide)
+    )
+    (property "Footprint" "" (at 119.38 111.76 0)
+      (effects (font (size 1.27 1.27)) hide)
+    )
+    (property "Datasheet" "" (at 119.38 111.76 0)
+      (effects (font (size 1.27 1.27)) hide)
+    )
+    (pin "~")
+    (instances
+      (project "hikari"
+        (path "/020af8ab-593e-45b9-b2cd-8db025796961/bb941b2b-0b73-4110-b4b0-cdc102f480d3"
+          (reference "#GND06") (unit 1)
+        )
+      )
+    )
+  )
   (symbol (lib_id "generic:GND") (at 104.14 119.38 0) (unit 1)
     (in_bom yes) (on_board yes) (dnp no) (fields_autoplaced)
@@
     )
   )
-  (symbol (lib_id "oscillators:xtal_osc") (at 138.43 113.03 0) (unit 1)
+  (symbol (lib_id "generic:R") (at 83.82 106.68 90) (unit 1)
+    (in_bom yes) (on_board yes) (dnp no)
+    (property "Reference" "R15" (at 85.09 106.68 90)
+      (effects (font (size 1.27 1.27)) (justify right top))
+    )
+    (property "Value" "5k1" (at 85.09 106.68 90)
+      (effects (font (size 1.27 1.27)) (justify right bottom))
+    )
+    (property "Footprint" "SMT:0603" (at 84.455 109.22 0)
+      (effects (font (size 1.27 1.27)) hide)
+    )
+    (property "Datasheet" "" (at 83.82 106.68 0)
+      (effects (font (size 1.27 1.27)) hide)
+    )
+    (pin "1")
+    (pin "2")
+    (instances
+      (project "hikari"
+        (path "/020af8ab-593e-45b9-b2cd-8db025796961/bb941b2b-0b73-4110-b4b0-cdc102f480d3"
+          (reference "R15") (unit 1)
+        )
+      )
+    )
+  )
+  (symbol (lib_id "oscillators:RH100-12.000-18-2020-EXT-TR") (at 138.43 113.03 0) (unit 1)
     (in_bom yes) (on_board yes) (dnp no) (fields_autoplaced)
     (property "Reference" "x1" (at 138.43 106.68 0)
       (effects (font (size 1.524 1.524)))
     )
-    (property "Value" "xtal_osc" (at 138.43 109.22 0)
+    (property "Value" "12MHZ" (at 138.43 109.22 0)
       (effects (font (size 1.524 1.524)))
     )
-    (property "Footprint" "" (at 138.43 111.76 0)
-      (effects (font (size 1.524 1.524)))
-    )
-    (property "Datasheet" "" (at 138.43 111.76 0)
-      (effects (font (size 1.524 1.524)))
+    (property "Footprint" "xtal:3.2x2.5CXO" (at 138.43 111.76 0)
+      (effects (font (size 1.524 1.524)) hide)
+    )
+    (property "Datasheet" "https://www.raltron.com/webproducts/specs/CRYSTAL/RH100-12.000-18-2020-EXT-TR.pdf" (at 138.43 111.76 0)
+      (effects (font (size 1.524 1.524)) hide)
+    )
+    (property "Digi-Key" "2151-RH100-12.000-18-2020-EXT-TRCT-ND" (at 138.43 113.03 0)
+      (effects (font (size 1.27 1.27)) hide)
     )
     (pin "1")
@@
         )
       )
+    )
+  )
+  (symbol (lib_id "generic:GND") (at 83.82 111.76 0) (unit 1)
+    (in_bom yes) (on_board yes) (dnp no) (fields_autoplaced)
+    (property "Reference" "#GND07" (at 87.63 110.49 0)
+      (effects (font (size 1.27 1.27)) hide)
+    )
+    (property "Value" "GND" (at 87.63 111.76 0)
+      (effects (font (size 1.27 1.27)) hide)
+    )
+    (property "Footprint" "" (at 83.82 111.76 0)
+      (effects (font (size 1.27 1.27)) hide)
+    )
+    (property "Datasheet" "" (at 83.82 111.76 0)
+      (effects (font (size 1.27 1.27)) hide)
+    )
+    (pin "~")
+    (instances
+      (project "hikari"
+        (path "/020af8ab-593e-45b9-b2cd-8db025796961/bb941b2b-0b73-4110-b4b0-cdc102f480d3"
+          (reference "#GND07") (unit 1)
+        )
+      )

Commit message: added Digi-Key part numbers to BOM
Parts:
- C13, C14: Digi-Key (none) -> 1276-1935-1-ND
- C15, C16: Digi-Key (none) -> 1292-1503-1-ND
- R13, R15: Digi-Key (none) -> 13-RC0603FR-135K1LCT-ND
Changed lines of the file:
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@@
+      (effects (font (size 1.27 1.27)) hide)
+    )
+    (property "Digi-Key" "13-RC0603FR-135K1LCT-ND" (at 119.38 106.68 0)
       (effects (font (size 1.27 1.27)) hide)
     )
@@
       (effects (font (size 1.27 1.27)) hide)
     )
+    (property "Digi-Key" "1276-1935-1-ND" (at 132.08 86.36 0)
+      (effects (font (size 1.27 1.27)) hide)
+    )
     (pin "1")
     (pin "2")
@@
     )
     (property "Datasheet" "" (at 83.82 106.68 0)
+      (effects (font (size 1.27 1.27)) hide)
+    )
+    (property "Digi-Key" "13-RC0603FR-135K1LCT-ND" (at 83.82 106.68 0)
       (effects (font (size 1.27 1.27)) hide)
     )
@@
       (effects (font (size 1.27 1.27)) hide)
     )
+    (property "Digi-Key" "1292-1503-1-ND" (at 129.54 118.11 0)
+      (effects (font (size 1.27 1.27)) hide)
+    )
     (pin "1")
     (pin "2")
@@
       (effects (font (size 1.27 1.27)) hide)
     )
+    (property "Digi-Key" "1276-1935-1-ND" (at 142.24 88.9 0)
+      (effects (font (size 1.27 1.27)) hide)
+    )
     (pin "1")
     (pin "2")
@@
       (effects (font (size 1.27 1.27)) hide)
     )
+    (property "Digi-Key" "1292-1503-1-ND" (at 147.32 118.11 0)
+      (effects (font (size 1.27 1.27)) hide)
+    )
