File: MCU.kicad_sch (KiCad schematic)
At the start: 12 parts, among them IC5 ESP-12F

Commit message: reviewn completed, fixes required
Other:
- note added: "GPIO 15PULLDOWN!!!"
Changed lines of the file:
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@@
     (effects (font (size 1.27 1.27)) (justify left bottom))
+  )
+  (text "GPIO 15PULLDOWN!!!" (at 111.76 137.16 0)
+    (effects (font (size 3 3) (thickness 0.6) bold (color 255 0 34 1)) (justify left bottom))
   )
   (label "temperature" (at 166.37 86.36 180) (fields_autoplaced)

Commit message: fixed errors, ready for order
Parts:
- added R17: 10k, SMT:0603, symbol generic:R
Connections:
- net GND: now also R17.1
- net at IC5.10 (IO15): now also R17.2
Other:
- note removed: "GPIO 15PULLDOWN!!!"
- moved on the sheet: R10, R11, R12, R9
